File: hardware/shack-interface/mcu.kicad_sch (KiCad schematic)
At the start: 15 parts, among them U3 TPS3823A-33, U4 74LVC1G74, U5 PCA9539, U61 USBLC6-2SC6

Commit message: Shack interface: end plates, schematic and PCB update; design log
Parts:
- added J15: DISPLAY, Connector_PinHeader_2.54mm:PinHeader_1x08_P2.54mm_Vertical, symbol Connector_Generic:Conn_01x08
Connections:
- net +3V3: now also J15.8 (Pin_8)
- net GND: now also J15.4 (Pin_4), J15.7 (Pin_7)
- net DISP_MOSI: now reaches A1.16 (IO9/BOOT)
- net DISP_MOSI: now also J15.6 (Pin_6)
- net DISP_SCK: now reaches A1.7 (IO2)
- net DISP_SCK: now also J15.5 (Pin_5)
- net LED_R1 renamed DISP_BL
- net DISP_BL: now also J15.1 (Pin_1)
- net LED_R2 renamed DISP_DC
- net DISP_DC: now also J15.3 (Pin_3)
- net LED_R3 renamed DISP_RST
- net DISP_RST: now also J15.2 (Pin_2)
- no-connect marks 15 -> 13
Other:
- note added: "Display J15 (D-180)"
