File: hardware/shack-interface/mcu.kicad_sch (KiCad schematic)
At the start: 16 parts, among them J15 DISPLAY, U3 TPS3823A-33, U4 74LVC1G74, U5 PCA9539, U61 USBLC6-2SC6

Commit message: Pre-order review; RF board seat keep-outs; part reuse P-1 to P-5
- docs/reviews/2026-10-31-pre-order-review.md: review of all three boards
  before ordering (verify scripts, ERC/DRC, pin maps, BOM, fab and case,
  firmware against spec, open items, part reuse).
- RF board (D-189, M-107): no other-net copper or vias under the case
  seats at S1 to S6 and the SO-239/SMA GND bosses; relay NC pads (pad 12)
  in netclass RF. Re-routed, DRC 0.
- Part reuse (D-190, M-108): one value text for 2k2, 100n 50V X7R and
  10n 50V X7R; shack PC817X order code as the controller; shack U4/U9 in
  VSSOP-8 (TI DCU, Nexperia DC) with fixed fan-out, re-routed.
  Netlists rf15, ctl15, si17; ERC 0.

Co-Authored-By: Claude Opus 5.5 <noreply@anthropic.com>
Parts:
- C64: value 100n 16V -> 100n 50V X7R
- U4: footprint Package_SO:SSOP-8_2.95x2.8mm_P0.65mm -> Package_SO:VSSOP-8_2.3x2mm_P0.5mm; MPN SN74LVC1G74DCTR -> SN74LVC1G74DCUR
Changed lines of the file:
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@@
 			)
 		)
-		(property "Footprint" "Package_SO:SSOP-8_2.95x2.8mm_P0.65mm"
+		(property "Footprint" "Package_SO:VSSOP-8_2.3x2mm_P0.5mm"
 			(at 304.8 68.58 0)
 			(hide yes)
@@
 			)
 		)
-		(property "Description" "D flip-flop, fault latch: D = GND, CLR_N = 3V3, PRE_N = RESET_N (TI SCES794G). Second source Nexperia 74LVC1G74DC"
+		(property "Description" "D flip-flop, fault latch: D = GND, CLR_N = 3V3, PRE_N = RESET_N (TI SCES794G, DCU VSSOP-8, D-190 as D-154). Second source Nexperia 74LVC1G74DC,125 (SOT765-1, same pin-out and MO-187 land)"
 			(at 304.8 68.58 0)
 			(hide yes)
@@
 			)
 		)
-		(property "MPN" "SN74LVC1G74DCTR"
+		(property "MPN" "SN74LVC1G74DCUR"
 			(at 304.8 68.58 0)
 			(hide yes)
@@
 			)
 		)
-		(property "Value" "100n 16V"
+		(property "Value" "100n 50V X7R"
 			(at 368.3 40.64 0)
 			(show_name no)

Commit message: S-2: SDA jumpers bridged 1-2 for RUST-1 by default
JP11 (controller) and JP61 (shack) use the Bridged12 solder jumper.
Pad 1 = SDA_IO10 (RUST-1), pad 3 = SDA_IO7 (RUST-2). Boards ship ready
for RUST-1; for RUST-2 cut 1-2 and bridge 2-3. New netlists ctl17 and
si18, new JP11/JP61 checks, boards re-routed, DRC clean. D-192, M-110.

Co-Authored-By: Claude Opus 5.5 <noreply@anthropic.com>
Parts:
- JP61: footprint Jumper:SolderJumper-3_P1.3mm_Open_RoundedPad1.0x1.5mm_NumberLabels -> Jumper:SolderJumper-3_P1.3mm_Bridged12_RoundedPad1.0x1.5mm_NumberLabels; symbol shack-interface:SolderJumper_3_Open -> shack-interface:SolderJumper_3_Bridged12
Connections:
- net SDA_IO10: now also JP61.1; no longer JP61.3
- net SDA_IO7: now also JP61.3; no longer JP61.1
Other:
- note added: "MCU: ESP32-C3 Rust board (A1) in two socket headers, the same module as the box (D-66). DevKit-RUST-1 Rev 1.2a fitted, RUST-2 also fits. Pads as the esp-rs Rust_Board footprint: left 1..16, right 28..17 top to bottom (D-93). SDA SEL JP61: 1-2 bridged by copper = RUST-1 (SDA IO10); RUST-2 (SDA IO7): cut 1-2, bridge 2-3 (D-94, D-192). Net labels at the DevKit pins; everything else is wired. 3V3 pin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"
- note removed: "MCU: ESP32-C3 Rust board (A1) in two socket headers, the same module as the box (D-66). DevKit-RUST-1 Rev 1.2a fitted, RUST-2 also fits. Pads as the esp-rs Rust_Board footprint: left 1..16, right 28..17 top to bottom (D-93). SDA SEL JP61: 2-3 RUST-1 (SDA IO10), 2-1 RUST-2 (SDA IO7) (D-94). Net labels at the DevKit pins; everything else is wired. 3V3 pin from the LD1117 (power sheet); EN low keeps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"
Changed lines of the file:
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@@
 			)
 		)
-		(property "Description" "ESP32-C3 Rust board pushed into gold-flash socket headers Sullins PPPC161LFBN-RC (1x16) and PPPC121LFBN-RC (1x12), rows 20.32 mm apart (D-55, D-66, D-93, D-95). RUST-1 Rev 1.2a fitted; RUST-2 fits with JP61 2-1"
+		(property "Description" "ESP32-C3 Rust board pushed into gold-flash socket headers Sullins PPPC161LFBN-RC (1x16) and PPPC121LFBN-RC (1x12), rows 20.32 mm apart (D-55, D-66, D-93, D-95). RUST-1 Rev 1.2a fitted; RUST-2 fits with JP61 1-2 cut and 2-3 bridged"
 			(at 101.6 170.18 0)
 			(hide yes)
@@
 	)
 	(symbol
-		(lib_id "shack-interface:SolderJumper_3_Open")
+		(lib_id "shack-interface:SolderJumper_3_Bridged12")
 		(at 274.32 121.92 270)
 		(unit 1)
@@
 			)
 		)
-		(property "Footprint" "Jumper:SolderJumper-3_P1.3mm_Open_RoundedPad1.0x1.5mm_NumberLabels"
+		(property "Footprint" "Jumper:SolderJumper-3_P1.3mm_Bridged12_RoundedPad1.0x1.5mm_NumberLabels"
 			(at 274.32 121.92 0)
 			(hide yes)
@@
 			)
 		)
-		(property "Description" "SDA select (D-94): bridge 2-3 for DevKit-RUST-1 (SDA GPIO10, pad 17), 2-1 for DevKit-RUST-2 (SDA GPIO7, pad 12). Firmware SDA pin must match"
+		(property "Description" "SDA select (D-94, D-192): 1-2 bridged by copper = DevKit-RUST-1 (SDA GPIO10, pad 17). DevKit-RUST-2 (SDA GPIO7, pad 12): cut 1-2, bridge 2-3. Firmware SDA pin must match"
 			(at 274.32 121.92 0)
 			(hide yes)
@@
 		)
 	)
-	(label "SDA_IO7"
+	(label "SDA_IO10"
 		(at 274.32 111.76 90)
 		(effects
@@
 		)
 	)
-	(label "SDA_IO10"
+	(label "SDA_IO7"
 		(at 274.32 132.08 270)
 		(effects
@@
 		)
 	)
-	(text "MCU: ESP32-C3 Rust board (A1) in two socket headers, the same module as the box (D-66). DevKit-RUST-1 Rev 1.2a fitted, RUST-2 also fits.\nPads as the esp-rs Rust_Board footprint: left 1..16, right 28..17 top to bottom (D-93). SDA SEL JP61: 2-3 RUST-1 (SDA IO10), 2-1 RUST-2 (SDA IO7) (D-94). Net labels at the DevKit pins; everything else is wired. 3V3 pin from the LD1117 (power sheet); EN low keeps the board buck off;\n5V not connected. USB-C to the Mac (Delock 64226) or the Pi (D-68).\nDirect GPIO (D-83): IO0 PERMIT_R1, IO1 WDI (kick at least every 0.9 s), IO3 LATCH_CLR (rising edge), IO4 PERMIT_R2, IO5 PERMIT_R3,\nIO6 DATA_TX, IO20 DATA_RX, IO21 SAFE_LOST (boot-ROM log pin, 1k series). SDA IO10 or IO7, SCL IO8 (board 10k pull-ups, SHTC3 0x70, IMU 0x68).\nIO2 DISP_SCK (WS2812 on the board sees only short pulses), IO9 DISP_MOSI (BOOT button: a press only disturbs the picture); both straps keep their pull-ups (D-180).\nBoard LED on IO7 (RUST-1) or IO10 (RUST-2): the SDA pin of the other board.\nFault latch (D-59): FAULT set at power-up, brown-out and watchdog time-out; cleared by a LATCH_CLR edge only when RESET_N is high.\nFAULT goes to the SAFE sheet and blocks every permit in hardware. RESET_N also resets the PCA9539: keys off, SW_STOP_N released.\nPCA9539 0x74 (D-92): IO0_0 SW_STOP_N (out), IO0_1 R1_TX, IO0_2 KEY_R1 (out), IO0_3 BAND_D, IO0_4 BAND_A, IO0_5 BAND_B, IO0_6 BAND_C,\nIO0_7 DISP_BL (out), IO1_0 KEY_R2 (out), IO1_1 R2_TX, IO1_2 DISP_DC (out), IO1_3 KEY_R3 (out), IO1_4 R3_TX, IO1_5 DISP_RST (out),\nIO1_6 KILL_S, IO1_7 LATCHED. Inputs not marked. Write outputs 0 before configuring (F1)."
+	(text "MCU: ESP32-C3 Rust board (A1) in two socket headers, the same module as the box (D-66). DevKit-RUST-1 Rev 1.2a fitted, RUST-2 also fits.\nPads as the esp-rs Rust_Board footprint: left 1..16, right 28..17 top to bottom (D-93). SDA SEL JP61: 1-2 bridged by copper = RUST-1 (SDA IO10); RUST-2 (SDA IO7): cut 1-2, bridge 2-3 (D-94, D-192). Net labels at the DevKit pins; everything else is wired. 3V3 pin from the LD1117 (power sheet); EN low keeps the board buck off;\n5V not connected. USB-C to the Mac (Delock 64226) or the Pi (D-68).\nDirect GPIO (D-83): IO0 PERMIT_R1, IO1 WDI (kick at least every 0.9 s), IO3 LATCH_CLR (rising edge), IO4 PERMIT_R2, IO5 PERMIT_R3,\nIO6 DATA_TX, IO20 DATA_RX, IO21 SAFE_LOST (boot-ROM log pin, 1k series). SDA IO10 or IO7, SCL IO8 (board 10k pull-ups, SHTC3 0x70, IMU 0x68).\nIO2 DISP_SCK (WS2812 on the board sees only short pulses), IO9 DISP_MOSI (BOOT button: a press only disturbs the picture); both straps keep their pull-ups (D-180).\nBoard LED on IO7 (RUST-1) or IO10 (RUST-2): the SDA pin of the other board.\nFault latch (D-59): FAULT set at power-up, brown-out and watchdog time-out; cleared by a LATCH_CLR edge only when RESET_N is high.\nFAULT goes to the SAFE sheet and blocks every permit in hardware. RESET_N also resets the PCA9539: keys off, SW_STOP_N released.\nPCA9539 0x74 (D-92): IO0_0 SW_STOP_N (out), IO0_1 R1_TX, IO0_2 KEY_R1 (out), IO0_3 BAND_D, IO0_4 BAND_A, IO0_5 BAND_B, IO0_6 BAND_C,\nIO0_7 DISP_BL (out), IO1_0 KEY_R2 (out), IO1_1 R2_TX, IO1_2 DISP_DC (out), IO1_3 KEY_R3 (out), IO1_4 R3_TX, IO1_5 DISP_RST (out),\nIO1_6 KILL_S, IO1_7 LATCHED. Inputs not marked. Write outputs 0 before configuring (F1)."
 		(exclude_from_sim no)
 		(at 25.4 22.86 0)

Commit message: S-10: MAX823SEUK+T first source, IRFL9014TRPBF-BE3 (D-195, M-118)
Supervisor U12 (controller), U3 and U6 (shack): MAX823SEUK+T first,
TPS3823A-33DBVR and APX823-29W5G-7 second. Same pin-out; RESET_N loads
are CMOS inputs; WDI and MR behave as the TPS3823 in our circuits.
RF Q1012 to Q1042: IRFL9014TRPBF-BE3. TLP176AM in stock at Mouser.
SO-239 83-798 stays single source, order first. Values and boards
unchanged. ERC 0 on all three.

Co-Authored-By: Claude Opus 5.5 <noreply@anthropic.com>
Parts:
- U3: MPN TPS3823A-33DBVR -> MAX823SEUK+T
Changed lines of the file:
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@@
 			)
 		)
-		(property "Description" "Supervisor 2.93 V + watchdog 0.9 to 2.5 s, push-pull RESET_N, -40 to 125 C (TI SLVS165O). A version"
+		(property "Description" "Supervisor 2.93 V (2.85 to 3.00) + watchdog 1.12 to 2.4 s, push-pull RESET_N (150 uA source: logic loads only), -40 to 125 C (ADI MAX823 19-0487 Rev 5). Second sources TI TPS3823A-33DBVR (A version only: no latch-up on WDI pulses during reset) and Diodes APX823-29W5G-7 (D-148, D-195)"
 			(at 269.24 66.04 0)
 			(hide yes)
@@
 			)
 		)
-		(property "MPN" "TPS3823A-33DBVR"
+		(property "MPN" "MAX823SEUK+T"
 			(at 269.24 66.04 0)
 			(hide yes)
@@
 			)
 		)
-		(property "Description" "WDI pull-down: a floating WDI would disable the watchdog (TPS3823 7.3.4)"
+		(property "Description" "WDI pull-down: a floating WDI would disable the watchdog (MAX823 WDI pin; TPS3823 7.3.4). MAX823 WDI sources max 20 uA: 20 mV low"
 			(at 251.46 67.31 0)
 			(hide yes)
