File: hardware/shack-interface/safe.kicad_sch (KiCad schematic)
At the start: 19 parts, among them U10 74LVC1G14, U11 74LVC1G02, U6 TPS3823A-33, U7 74LVC1G14, U8 74LVC1G08, U9 74LVC1G74

Commit message: Shack interface: end plates, schematic and PCB update; design log
Parts:
- R75: value 10k -> 2k2
Changed lines of the file:
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@@
 			)
 		)
-		(property "Value" "10k"
+		(property "Value" "2k2"
 			(at 41.91 163.83 0)
 			(show_name no)
@@
 			)
 		)
-		(property "Description" "KILL_S pull-up: open (KILL pressed or switch unplugged) reads high"
+		(property "Description" "KILL_S pull-up: open (KILL pressed or switch unplugged) reads high. 2k2 gives 1.5 mA, above the 1 mA contact minimum of the EAO 84 (D-181)"
 			(at 40.64 161.29 0)
 			(hide yes)
