File: hardware/shack-interface/power.kicad_sch (KiCad schematic)
At the start: 17 parts, among them U1 L7805CV, U2 LD1117S33CTR

Commit message: Pre-order review; RF board seat keep-outs; part reuse P-1 to P-5
- docs/reviews/2026-10-31-pre-order-review.md: review of all three boards
  before ordering (verify scripts, ERC/DRC, pin maps, BOM, fab and case,
  firmware against spec, open items, part reuse).
- RF board (D-189, M-107): no other-net copper or vias under the case
  seats at S1 to S6 and the SO-239/SMA GND bosses; relay NC pads (pad 12)
  in netclass RF. Re-routed, DRC 0.
- Part reuse (D-190, M-108): one value text for 2k2, 100n 50V X7R and
  10n 50V X7R; shack PC817X order code as the controller; shack U4/U9 in
  VSSOP-8 (TI DCU, Nexperia DC) with fixed fan-out, re-routed.
  Netlists rf15, ctl15, si17; ERC 0.

Co-Authored-By: Claude Opus 5.5 <noreply@anthropic.com>
Parts:
- C3: value 100n -> 100n 50V X7R
Changed lines of the file:
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@@
 			)
 		)
-		(property "Value" "100n"
+		(property "Value" "100n 50V X7R"
 			(at 142.49 58.42 0)
 			(show_name no)
