File: hardware/shack-interface/shack-interface.kicad_pcb (KiCad board)
At the start: 4 copper layers, 160 x 161 mm, 290 parts, among them J1 RJ45 LINK, J11 R1 mini-DIN, J12 R2 mini-DIN, J13 R3 mini-DIN, J14 USB4105-GF-A, J15 DISPLAY, J2 KILL switch, J3 13.8 V IN, J6 Front panel, J7 KILL state, Q11 BCP53-16, Q12 BC857B, Q13 BSS138BK, Q21 BCP53-16, Q22 BC857B, Q23 BSS138BK, Q31 BCP53-16, Q32 BC857B, Q33 BSS138BK, Q34 BC847B, Q41 BCP53-16, Q42 BC857B, Q44 BC847B, U1 L7805CV, U10 74LVC1G14, U11 74LVC1G02, U2 LD1117S33CTR, U201 74LVC1G08, U202 74LVC1G08, U203 TLP4176G, U204 TLP176AM, U205 PC817X, U3 TPS3823A-33, U301 74LVC1G08, U302 74LVC1G08, U303 TLP4176G, U304 TLP176AM, U305 PC817X, U4 74LVC1G74, U401 74LVC1G08, U402 74LVC1G08, U403 TLP4176G, U404 TLP176AM, U405 PC817X, U5 PCA9539, U6 TPS3823A-33, U61 USBLC6-2SC6, U7 74LVC1G14, U8 74LVC1G08, U9 74LVC1G74

Commit message: S-2: SDA jumpers bridged 1-2 for RUST-1 by default
JP11 (controller) and JP61 (shack) use the Bridged12 solder jumper.
Pad 1 = SDA_IO10 (RUST-1), pad 3 = SDA_IO7 (RUST-2). Boards ship ready
for RUST-1; for RUST-2 cut 1-2 and bridge 2-3. New netlists ctl17 and
si18, new JP11/JP61 checks, boards re-routed, DRC clean. D-192, M-110.

Co-Authored-By: Claude Opus 5.5 <noreply@anthropic.com>
Parts:
- JP61: footprint Jumper:SolderJumper-3_P1.3mm_Open_RoundedPad1.0x1.5mm_NumberLabels -> Jumper:SolderJumper-3_P1.3mm_Bridged12_RoundedPad1.0x1.5mm_NumberLabels
- turned JP61 to -90 degrees
Connections:
- JP61 pad 1: /MCU and expander/SDA_IO7 -> /MCU and expander/SDA_IO10
- JP61 pad 3: /MCU and expander/SDA_IO10 -> /MCU and expander/SDA_IO7
Routing:
- net /Link to the box/L1N: track 59.5 -> 41.0 mm, vias 7 -> 6
- net +3V3: track 671.9 -> 662.7 mm, vias 60 -> 67
- net /MCU and expander/SAFE_LOST: track 103.1 -> 109.3 mm
- net /Radio port R1/TX_EN: track 151.1 -> 156.8 mm
- net /Link to the box/R1_TX: track 106.6 -> 111.8 mm
- net /MCU and expander/KILL_S: track 153.7 -> 158.5 mm
- net /SAFE latch/RESET_CLK: track 15.4 -> 19.7 mm, vias 2 -> 4
- net /Link to the box/L4N: track 29.7 -> 34.0 mm, vias 4 -> 5
- net /Link to the box/L2N: track 34.8 -> 30.7 mm
- net +13V8: track 289.3 -> 293.2 mm
- net /MCU and expander/DISP_MOSI: track 64.7 -> 61.4 mm, vias 3 -> 1
- net /MCU and expander/LATCH_CLR: track 39.1 -> 41.5 mm, vias 3 -> 4
- net Net-(D43-K): track 12.0 -> 14.4 mm
- net Net-(Q21-B): track 21.3 -> 19.4 mm, vias 5 -> 2
- net Net-(Q31-E): track 12.1 -> 10.1 mm
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Other:
- board text added: "Shack interface rev A (p8d)"
- board text removed: "Shack interface rev A (p8c)"
