File: hardware/shack-interface/shack-interface.kicad_pcb (KiCad board)
At the start: 4 copper layers, 160 x 161 mm, 290 parts, among them J1 RJ45 LINK, J11 R1 mini-DIN, J12 R2 mini-DIN, J13 R3 mini-DIN, J14 USB4105-GF-A, J15 DISPLAY, J2 KILL switch, J3 13.8 V IN, J6 Front panel, J7 KILL state, Q11 BCP53-16, Q12 BC857B, Q13 BSS138BK, Q21 BCP53-16, Q22 BC857B, Q23 BSS138BK, Q31 BCP53-16, Q32 BC857B, Q33 BSS138BK, Q34 BC847B, Q41 BCP53-16, Q42 BC857B, Q44 BC847B, U1 L7805CV, U10 74LVC1G14, U11 74LVC1G02, U2 LD1117S33CTR, U201 74LVC1G08, U202 74LVC1G08, U203 TLP4176G, U204 TLP176AM, U205 PC817X, U3 TPS3823A-33, U301 74LVC1G08, U302 74LVC1G08, U303 TLP4176G, U304 TLP176AM, U305 PC817X, U4 74LVC1G74, U401 74LVC1G08, U402 74LVC1G08, U403 TLP4176G, U404 TLP176AM, U405 PC817X, U5 PCA9539, U6 TPS3823A-33, U61 USBLC6-2SC6, U7 74LVC1G14, U8 74LVC1G08, U9 74LVC1G74

Commit message: S-8: shack interface 159.6 mm wide
The side edges in the extrusion slots move in 0.2 mm each (x 0.2 and
159.8), so the board fits the 160 mm slots with the JLC outline
tolerance. Centre stays at x 80: end plates unchanged. Shack layout
p8e: 155/155 nets, 429 vias; DRC as p8d plus one starved thermal
(R418 pad 2); JP406 reference hidden. D-194, M-112.

Co-Authored-By: Claude Opus 5.5 <noreply@anthropic.com>
Routing:
- net /Link to the box/KILL_2: track 105.0 -> 111.7 mm, vias 4 -> 6
- net /MCU and expander/SAFE_LOST: track 109.3 -> 103.2 mm
- net +3V3: track 662.7 -> 667.2 mm, vias 67 -> 61
- net /Radio port R1/TX_EN: track 156.8 -> 152.6 mm, vias 8 -> 6
- net /MCU and expander/KILL_S: track 158.5 -> 154.4 mm
- net /Link to the box/L4N: track 34.0 -> 38.0 mm, vias 5 -> 6
- net +13V8: track 293.2 -> 297.1 mm, vias 28 -> 27
- net Net-(D21-A2): track 30.6 -> 34.3 mm, vias 3 -> 4
- net /Link to the box/KILL_1: track 86.4 -> 89.9 mm, vias 9 -> 5
- net /MCU and expander/DISP_MOSI: track 61.4 -> 64.7 mm, vias 1 -> 3
- net Net-(D33-K): track 11.7 -> 14.5 mm
- net /MCU and expander/USB_DP: track 163.9 -> 161.2 mm, vias 5 -> 7
- net Net-(D31-A1): track 54.5 -> 56.9 mm, vias 4 -> 2
- net /MCU and expander/SDA: track 65.8 -> 68.0 mm
- net /Radio port R2/DIN2: track 56.7 -> 58.9 mm, vias 3 -> 1
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Other:
- board size 160 x 161 mm -> 159.6 x 161 mm
- board text added: "Shack interface rev A (p8e)"
- board text removed: "Shack interface rev A (p8d)"
