File: hardware/shack-interface/link.kicad_sch (KiCad schematic)
At the start: 60 parts, among them Q11 BCP53-16, Q12 BC857B, Q13 BSS138BK, Q21 BCP53-16, Q22 BC857B, Q23 BSS138BK, Q31 BCP53-16, Q32 BC857B, Q33 BSS138BK, Q34 BC847B, Q41 BCP53-16, Q42 BC857B, Q44 BC847B

Commit message: S-4: MPN BSS138BK,215 (Nexperia) on RF and shack (M-115)
The ROHM BSS138BKT116 has the same name and another pin order. All 45
BSS138BK (RF 42, shack 3) now carry MPN BSS138BK,215. Nexperia pinning
1 G, 2 S, 3 D matches the footprint. ERC 0 on both; boards and
netlists unchanged.

Co-Authored-By: Claude Opus 5.5 <noreply@anthropic.com>
Parts:
- Q13, Q23, Q33: MPN BSS138BK -> BSS138BK,215
Changed lines of the file:
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@@
 			)
 		)
-		(property "MPN" "BSS138BK"
+		(property "MPN" "BSS138BK,215"
 			(at 109.22 53.34 0)
 			(hide yes)
@@
 			)
 		)
-		(property "MPN" "BSS138BK"
+		(property "MPN" "BSS138BK,215"
 			(at 109.22 116.84 0)
 			(hide yes)
@@
 			)
 		)
-		(property "MPN" "BSS138BK"
+		(property "MPN" "BSS138BK,215"
 			(at 109.22 180.34 0)
 			(hide yes)
