File: hardware/shack-interface/radioport.kicad_sch (KiCad schematic)
At the start: 56 parts, among them U201 74LVC1G08, U202 74LVC1G08, U203 TLP4176G, U204 TLP176AM, U205 PC817X

Commit message: Pre-order review; RF board seat keep-outs; part reuse P-1 to P-5
- docs/reviews/2026-10-31-pre-order-review.md: review of all three boards
  before ordering (verify scripts, ERC/DRC, pin maps, BOM, fab and case,
  firmware against spec, open items, part reuse).
- RF board (D-189, M-107): no other-net copper or vias under the case
  seats at S1 to S6 and the SO-239/SMA GND bosses; relay NC pads (pad 12)
  in netclass RF. Re-routed, DRC 0.
- Part reuse (D-190, M-108): one value text for 2k2, 100n 50V X7R and
  10n 50V X7R; shack PC817X order code as the controller; shack U4/U9 in
  VSSOP-8 (TI DCU, Nexperia DC) with fixed fan-out, re-routed.
  Netlists rf15, ctl15, si17; ERC 0.

Co-Authored-By: Claude Opus 5.5 <noreply@anthropic.com>
Parts:
- U205: MPN PC817X -> PC817X2NSZ9F
Changed lines of the file:
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@@
 			)
 		)
-		(property "MPN" "PC817X"
+		(property "MPN" "PC817X2NSZ9F"
 			(at 101.6 119.38 0)
 			(hide yes)

Commit message: S-6: order codes for LM2901, JST XH and shack 1 nF (M-117)
MPN fields only: RF U801 LM2901DR; shack J2/J7 B2B-XH-A(LF)(SN),
J6 B4B-XH-A(LF)(SN), 21 x 1 nF C0G GRM1885C1H102JA01D. Values,
netlists and boards unchanged. ERC 0 on both.

Co-Authored-By: Claude Opus 5.5 <noreply@anthropic.com>
Parts:
- C211, C212, C213, C214, C216, C217, C218: MPN (none) -> GRM1885C1H102JA01D
Changed lines of the file:
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@@
 			)
 		)
+		(property "MPN" "GRM1885C1H102JA01D"
+			(at 353.06 82.55 0)
+			(hide yes)
+			(show_name no)
+			(do_not_autoplace no)
+			(effects
+				(font
+					(size 1.27 1.27)
+				)
+				(justify left)
+			)
+		)
 		(pin "1"
 		)
@@
 			)
 		)
+		(property "MPN" "GRM1885C1H102JA01D"
+			(at 353.06 67.31 0)
+			(hide yes)
+			(show_name no)
+			(do_not_autoplace no)
+			(effects
+				(font
+					(size 1.27 1.27)
+				)
+				(justify left)
+			)
+		)
 		(pin "1"
 		)
@@
 			)
 		)
+		(property "MPN" "GRM1885C1H102JA01D"
+			(at 353.06 52.07 0)
+			(hide yes)
+			(show_name no)
+			(do_not_autoplace no)
+			(effects
+				(font
+					(size 1.27 1.27)
+				)
+				(justify left)
+			)
+		)
 		(pin "1"
 		)
@@
 			)
 		)
+		(property "MPN" "GRM1885C1H102JA01D"
+			(at 353.06 123.19 0)
+			(hide yes)
+			(show_name no)
+			(do_not_autoplace no)
+			(effects
+				(font
+					(size 1.27 1.27)
+				)
+				(justify left)
+			)
+		)
 		(pin "1"
 		)
@@
 			)
 		)
+		(property "MPN" "GRM1885C1H102JA01D"
+			(at 353.06 161.29 0)
+			(hide yes)
+			(show_name no)
+			(do_not_autoplace no)
+			(effects
+				(font
+					(size 1.27 1.27)
+				)
+				(justify left)
+			)
+		)
 		(pin "1"
 		)
@@
 			)
 		)
+		(property "MPN" "GRM1885C1H102JA01D"
+			(at 353.06 194.31 0)
+			(hide yes)
+			(show_name no)
+			(do_not_autoplace no)
+			(effects
+				(font
+					(size 1.27 1.27)
+				)
+				(justify left)
+			)
+		)
 		(pin "1"
 		)
@@
 			(at 353.06 214.63 0)
 			(hide yes)
+			(show_name no)
+			(do_not_autoplace no)
+			(effects
+				(font
+					(size 1.27 1.27)
+				)
+				(justify left)
+			)
+		)
+		(property "MPN" "GRM1885C1H102JA01D"
+			(at 353.06 214.63 0)
+			(hide yes)
