File: hardware/shack-interface/shack-interface.kicad_sch (KiCad schematic)
At the start: 10 parts, among them J1 RJ45 LINK, J11 R1 mini-DIN, J12 R2 mini-DIN, J13 R3 mini-DIN, J14 USB4105-GF-A, J2 KILL switch, J3 13.8 V IN, J6 Front panel, J7 KILL state

Commit message: S-6: order codes for LM2901, JST XH and shack 1 nF (M-117)
MPN fields only: RF U801 LM2901DR; shack J2/J7 B2B-XH-A(LF)(SN),
J6 B4B-XH-A(LF)(SN), 21 x 1 nF C0G GRM1885C1H102JA01D. Values,
netlists and boards unchanged. ERC 0 on both.

Co-Authored-By: Claude Opus 5.5 <noreply@anthropic.com>
Parts:
- J2, J7: MPN (none) -> B2B-XH-A(LF)(SN)
- J6: MPN (none) -> B4B-XH-A(LF)(SN)
Changed lines of the file:
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@@
+			)
+		)
+		(property "MPN" "B2B-XH-A(LF)(SN)"
+			(at 83.82 81.28 0)
+			(hide yes)
+			(show_name no)
+			(do_not_autoplace no)
+			(effects
+				(font
+					(size 1.27 1.27)
+				)
+				(justify left)
 			)
 		)
@@
 			)
 		)
+		(property "MPN" "B2B-XH-A(LF)(SN)"
+			(at 231.14 114.3 0)
+			(hide yes)
+			(show_name no)
+			(do_not_autoplace no)
+			(effects
+				(font
+					(size 1.27 1.27)
+				)
+				(justify left)
+			)
+		)
 		(pin "1"
 		)
@@
 			(at 304.8 60.96 0)
 			(hide yes)
+			(show_name no)
+			(do_not_autoplace no)
+			(effects
+				(font
+					(size 1.27 1.27)
+				)
+				(justify left)
+			)
+		)
+		(property "MPN" "B4B-XH-A(LF)(SN)"
+			(at 304.8 60.96 0)
+			(hide yes)
