File: hardware/shack-interface/endplates/rear-panel.kicad_pcb (KiCad board)
At the start: 2 copper layers, 165 x 51.1 mm, 4 parts

Commit message: Shack interface: end plates, schematic and PCB update; design log
Other:
- board text added: "SRM shack interface rear plate rev A (a3) 2026-10"
- board text removed: "SRM shack interface rear plate rev A (a1) 2026-10"
Changed lines of the file:
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@@
+	(footprint "MountingHole_3.7mm_Pad"
+		(layer "F.Cu")
+		(at 180.262 23.81)
+		(descr "Mounting Hole 3.7mm, generated by kicad-footprint-generator mountinghole.py")
+		(tags "mountinghole")
+		(property "Reference" "REF**"
+			(at 0 -4.65 0)
+			(layer "F.SilkS")
+			(hide yes)
+			(effects
+				(font
+					(size 1 1)
+					(thickness 0.15)
+				)
+			)
+		)
+		(property "Value" "MountingHole_3.7mm_Pad"
+			(at 0 4.65 0)
+			(layer "F.Fab")
+			(hide yes)
+			(effects
+				(font
+					(size 1 1)
+					(thickness 0.15)
+				)
+			)
+		)
+		(property "Datasheet" ""
+			(at 0 0 0)
+			(layer "F.Fab")
+			(hide yes)
+			(effects
+				(font
+					(size 1.27 1.27)
+				)
+			)
+		)
+		(property "Description" ""
+			(at 0 0 0)
+			(layer "F.Fab")
+			(hide yes)
+			(effects
+				(font
+					(size 1.27 1.27)
+				)
+			)
+		)
+		(property "KiLib_Generator" "mounting_hardware/mounting_hole"
+			(at 0 0 0)
+			(layer "F.SilkS")
+			(hide yes)
+			(effects
+				(font
+					(size 1 1)
+					(thickness 0.15)
+				)
+			)
+		)
+		(attr exclude_from_pos_files exclude_from_bom)
+		(duplicate_pad_numbers_are_jumpers no)
+		(fp_circle
+			(center 0 0)
+			(end 3.7 0)
+			(stroke
+				(width 0.15)
+				(type solid)
+			)
+			(fill no)
+			(layer "Cmts.User")
+		)
+		(fp_circle
+			(center 0 0)
+			(end 3.95 0)
+			(stroke
+				(width 0.05)
+				(type solid)
+			)
+			(fill no)
+			(layer "F.CrtYd")
+		)
+		(fp_text user "${REFERENCE}"
+			(at 0 0 0)
+			(layer "F.Fab")
+			(effects
+				(font
+					(size 1 1)
+					(thickness 0.15)
+				)
+			)
+		)
+		(pad "1" thru_hole circle
+			(at 0 0)
+			(size 6 6)
+			(drill 3.7)
+			(layers "*.Cu" "*.Mask")
+			(remove_unused_layers no)
+			(net "CHASSIS")
+			(zone_connect 2)
+		)
+		(embedded_fonts no)
+	)
 	(footprint "MountingHole_3.7mm_Pad"
 		(layer "F.Cu")
@@
 	(footprint "MountingHole_3.7mm_Pad"
 		(layer "F.Cu")
-		(at 24.738 23.81)
+		(at 180.262 67.32)
 		(descr "Mounting Hole 3.7mm, generated by kicad-footprint-generator mountinghole.py")
 		(tags "mountinghole")
@@
 	(footprint "MountingHole_3.7mm_Pad"
 		(layer "F.Cu")
-		(at 180.262 23.81)
+		(at 24.738 23.81)
 		(descr "Mounting Hole 3.7mm, generated by kicad-footprint-generator mountinghole.py")
 		(tags "mountinghole")
@@
 		(embedded_fonts no)
 	)
-	(footprint "MountingHole_3.7mm_Pad"
-		(layer "F.Cu")
-		(at 180.262 67.32)
-		(descr "Mounting Hole 3.7mm, generated by kicad-footprint-generator mountinghole.py")
-		(tags "mountinghole")
-		(property "Reference" "REF**"
-			(at 0 -4.65 0)
-			(layer "F.SilkS")
-			(hide yes)
-			(effects
-				(font
-					(size 1 1)
-					(thickness 0.15)
-				)
-			)
-		)
-		(property "Value" "MountingHole_3.7mm_Pad"
-			(at 0 4.65 0)
-			(layer "F.Fab")
-			(hide yes)
-			(effects
-				(font
-					(size 1 1)
-					(thickness 0.15)
-				)
-			)
-		)
-		(property "Datasheet" ""
-			(at 0 0 0)
-			(layer "F.Fab")
-			(hide yes)
-			(effects
-				(font
-					(size 1.27 1.27)
-				)
-			)
-		)
-		(property "Description" ""
-			(at 0 0 0)
-			(layer "F.Fab")
-			(hide yes)
-			(effects
-				(font
-					(size 1.27 1.27)
-				)
-			)
-		)
-		(property "KiLib_Generator" "mounting_hardware/mounting_hole"
-			(at 0 0 0)
-			(layer "F.SilkS")
-			(hide yes)
-			(effects
-				(font
-					(size 1 1)
-					(thickness 0.15)
-				)
-			)
-		)
-		(attr exclude_from_pos_files exclude_from_bom)
-		(duplicate_pad_numbers_are_jumpers no)
-		(fp_circle
-			(center 0 0)
-			(end 3.7 0)
-			(stroke
-				(width 0.15)
-				(type solid)
-			)
-			(fill no)
-			(layer "Cmts.User")
-		)
-		(fp_circle
-			(center 0 0)
-			(end 3.95 0)
-			(stroke
-				(width 0.05)
-				(type solid)
-			)
-			(fill no)
-			(layer "F.CrtYd")
-		)
-		(fp_text user "${REFERENCE}"
-			(at 0 0 0)
-			(layer "F.Fab")
-			(effects
-				(font
-					(size 1 1)
-					(thickness 0.15)
-				)
-			)
-		)
-		(pad "1" thru_hole circle
-			(at 0 0)
-			(size 6 6)
-			(drill 3.7)
-			(layers "*.Cu" "*.Mask")
-			(remove_unused_layers no)
-			(net "CHASSIS")
-			(zone_connect 2)
-		)
-		(embedded_fonts no)
-	)
 	(gr_arc
 		(start 20 23.9)
@@
 		)
 	)
-	(gr_text "SRM shack interface rear plate  rev A (a1)  2026-10"
+	(gr_text "SRM shack interface rear plate  rev A (a3)  2026-10"
 		(at 102.5 63.13 0)
 		(layer "B.SilkS")
