File: hardware/unit/rf-board/rf-board.kicad_pcb (KiCad board)
At the start: 6 copper layers, 268 x 230 mm, 357 parts, among them J1 83-798 SO-239, J10 83-798 SO-239, J11 XT60PW-M, J12 XT60PW-M, J13 XT30PW-M, J14 Controller header, J2 83-798 SO-239, J3 83-798 SO-239, J4 SMA jack EXP, J5 SMA jack EXP, J6 SMA jack EXP, J7 83-798 SO-239, J8 83-798 SO-239, J9 83-798 SO-239, K101 RTD14012F, K102 RTD14012F, K103 RTD14012F, K104 RTD14012F, K105 RTD14012F, K106 RTD14012F, K107 RTD14012F, K108 RTD14012F, K109 RTD14012F, K110 RTD14012F, K111 RTD14012F, K201 RTD14012F, K202 RTD14012F, K203 RTD14012F, K204 RTD14012F, K205 RTD14012F, K206 RTD14012F, K207 RTD14012F, K208 RTD14012F, K209 RTD14012F, K210 RTD14012F, K211 RTD14012F, K301 RTD14012F, K302 RTD14012F, K303 RTD14012F, K304 RTD14012F, K305 RTD14012F, K306 RTD14012F, K307 RTD14012F, K308 RTD14012F, K309 RTD14012F, K310 RTD14012F, K311 RTD14012F, K401 RTD14012F, K501 RTD14012F, K601 RTD14012F, K701 RTD14012F, Q1 PMV50EPEA, Q101 BSS138BK, Q1011 BC857B, Q1012 IRFL9014, Q1013 BSS138BK, Q102 BSS138BK, Q1021 BC857B, Q1022 IRFL9014, Q1023 BSS138BK, Q103 BSS138BK, Q1031 BC857B, Q1032 IRFL9014, Q1033 BSS138BK, Q104 BSS138BK, Q1041 BC857B, Q1042 IRFL9014, Q1043 BSS138BK, Q105 BSS138BK, Q106 BSS138BK, Q107 BSS138BK, Q108 BSS138BK, Q109 BSS138BK, Q110 BSS138BK, Q111 BSS138BK, Q2 BSS138BK, Q201 BSS138BK, Q202 BSS138BK, Q203 BSS138BK, Q204 BSS138BK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

Commit message: Pre-order review; RF board seat keep-outs; part reuse P-1 to P-5
- docs/reviews/2026-10-31-pre-order-review.md: review of all three boards
  before ordering (verify scripts, ERC/DRC, pin maps, BOM, fab and case,
  firmware against spec, open items, part reuse).
- RF board (D-189, M-107): no other-net copper or vias under the case
  seats at S1 to S6 and the SO-239/SMA GND bosses; relay NC pads (pad 12)
  in netclass RF. Re-routed, DRC 0.
- Part reuse (D-190, M-108): one value text for 2k2, 100n 50V X7R and
  10n 50V X7R; shack PC817X order code as the controller; shack U4/U9 in
  VSSOP-8 (TI DCU, Nexperia DC) with fixed fan-out, re-routed.
  Netlists rf15, ctl15, si17; ERC 0.

Co-Authored-By: Claude Opus 5.5 <noreply@anthropic.com>
Parts:
- C1011, C1021, C1031, C1041, C801: value 100n -> 100n 50V X7R
- C4: value 10n -> 10n 50V X7R
- R2, R901, R902: value 2.2k -> 2k2
Routing:
- net Net-(D207-A): track 168.7 -> 101.5 mm, vias 5 -> 3
- net Net-(D302-A): track 192.0 -> 131.3 mm, vias 6 -> 5
- net /R2_RX4_DRV: track 214.0 -> 270.5 mm, vias 4 -> 9
- net /R2_TX4_DRV: track 220.4 -> 276.1 mm, vias 4 -> 8
- net CLAMP_RLY: track 196.0 -> 251.6 mm, vias 4 -> 7
- net /R1_RX4_DRV: track 223.1 -> 275.3 mm, vias 2 -> 9
- net /RLY_EN: track 456.4 -> 503.3 mm, vias 18 -> 31
- net /A2_K1_DRV: track 236.7 -> 194.3 mm, vias 14 -> 7
- net /R3_RX3_DRV: track 232.6 -> 191.0 mm, vias 10 -> 7
- net +5V: track 343.5 -> 382.8 mm, vias 14 -> 18
- net /A3_K1_DRV: track 261.4 -> 227.1 mm, vias 9 -> 8
- net +3V3: track 614.4 -> 643.3 mm, vias 31 -> 43
- net +12V_SW: track 1189.2 -> 1160.4 mm, vias 95 -> 89
- net /A2_RFDET: track 333.1 -> 305.6 mm, vias 15 -> 12
- net /R3_TX3_DRV: track 215.4 -> 188.2 mm, vias 13 -> 6
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Other:
- board text added: "RF board rev C (p3-keep)"
- board text removed: "RF board rev C (p3-silk)"
