File: hardware/unit/rf-board/antenna_port.kicad_sch (KiCad schematic)
At the start: 15 parts, among them K401 RTD14012F, Q401 BSS138BK

Commit message: S-4: MPN BSS138BK,215 (Nexperia) on RF and shack (M-115)
The ROHM BSS138BKT116 has the same name and another pin order. All 45
BSS138BK (RF 42, shack 3) now carry MPN BSS138BK,215. Nexperia pinning
1 G, 2 S, 3 D matches the footprint. ERC 0 on both; boards and
netlists unchanged.

Co-Authored-By: Claude Opus 5.5 <noreply@anthropic.com>
Parts:
- Q401: MPN BSS138BK -> BSS138BK,215
Changed lines of the file:
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@@
 			)
 		)
-		(property "MPN" "BSS138BK"
+		(property "MPN" "BSS138BK,215"
 			(at 149.86 116.84 0)
 			(hide yes)
