File: hardware/unit/rf-board/radio_port.kicad_sch (KiCad schematic)
At the start: 45 parts, among them K101 RTD14012F, K102 RTD14012F, K103 RTD14012F, K104 RTD14012F, K105 RTD14012F, K106 RTD14012F, K107 RTD14012F, K108 RTD14012F, K109 RTD14012F, K110 RTD14012F, K111 RTD14012F, Q101 BSS138BK, Q102 BSS138BK, Q103 BSS138BK, Q104 BSS138BK, Q105 BSS138BK, Q106 BSS138BK, Q107 BSS138BK, Q108 BSS138BK, Q109 BSS138BK, Q110 BSS138BK, Q111 BSS138BK

Commit message: S-4: MPN BSS138BK,215 (Nexperia) on RF and shack (M-115)
The ROHM BSS138BKT116 has the same name and another pin order. All 45
BSS138BK (RF 42, shack 3) now carry MPN BSS138BK,215. Nexperia pinning
1 G, 2 S, 3 D matches the footprint. ERC 0 on both; boards and
netlists unchanged.

Co-Authored-By: Claude Opus 5.5 <noreply@anthropic.com>
Parts:
- Q101, Q102, Q103, Q104, Q105, Q106, Q107, Q108, Q109, Q110, Q111: MPN BSS138BK -> BSS138BK,215
Changed lines of the file:
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@@
 			)
 		)
-		(property "MPN" "BSS138BK"
+		(property "MPN" "BSS138BK,215"
 			(at 73.66 238.76 0)
 			(hide yes)
@@
 			)
 		)
-		(property "MPN" "BSS138BK"
+		(property "MPN" "BSS138BK,215"
 			(at 93.98 96.52 0)
 			(hide yes)
@@
 			)
 		)
-		(property "MPN" "BSS138BK"
+		(property "MPN" "BSS138BK,215"
 			(at 144.78 96.52 0)
 			(hide yes)
@@
 			)
 		)
-		(property "MPN" "BSS138BK"
+		(property "MPN" "BSS138BK,215"
 			(at 195.58 96.52 0)
 			(hide yes)
@@
 			)
 		)
-		(property "MPN" "BSS138BK"
+		(property "MPN" "BSS138BK,215"
 			(at 246.38 96.52 0)
 			(hide yes)
@@
 			)
 		)
-		(property "MPN" "BSS138BK"
+		(property "MPN" "BSS138BK,215"
 			(at 297.18 96.52 0)
 			(hide yes)
@@
 			)
 		)
-		(property "MPN" "BSS138BK"
+		(property "MPN" "BSS138BK,215"
 			(at 93.98 172.72 0)
 			(hide yes)
@@
 			)
 		)
-		(property "MPN" "BSS138BK"
+		(property "MPN" "BSS138BK,215"
 			(at 144.78 172.72 0)
 			(hide yes)
@@
 			)
 		)
-		(property "MPN" "BSS138BK"
+		(property "MPN" "BSS138BK,215"
 			(at 195.58 172.72 0)
 			(hide yes)
@@
 			)
 		)
-		(property "MPN" "BSS138BK"
+		(property "MPN" "BSS138BK,215"
 			(at 246.38 172.72 0)
 			(hide yes)
@@
 			)
 		)
-		(property "MPN" "BSS138BK"
+		(property "MPN" "BSS138BK,215"
 			(at 297.18 172.72 0)
 			(hide yes)
