File: hardware/unit/rf-board/rf-board.kicad_sch (KiCad schematic)
At the start: 14 parts, among them J1 83-798 SO-239, J10 83-798 SO-239, J11 XT60PW-M, J12 XT60PW-M, J13 XT30PW-M, J14 Controller header, J2 83-798 SO-239, J3 83-798 SO-239, J4 SMA jack EXP, J5 SMA jack EXP, J6 SMA jack EXP, J7 83-798 SO-239, J8 83-798 SO-239, J9 83-798 SO-239

Commit message: S-5: RF J14 = Samtec TSW-112-07-L-D (M-116)
Post 5.84 mm above the body, 10 uin gold on the post. Mates with the
ESQ-112-33-G-D socket: engagement 4.89 mm at the 19.7 mm board gap,
inside 3.68 to 6.35 mm. ERC 0; boards unchanged.

Co-Authored-By: Claude Opus 5.5 <noreply@anthropic.com>
Parts:
- J14: MPN (none) -> TSW-112-07-L-D
Changed lines of the file:
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@@
 			)
 		)
-		(property "Description" "Board-to-board header. Unit 1: controller board (MCU, RJ45 LINK). Unit 2: EXP ribbon from the unit 1 controller board, +5V pins open at the controller end. 3.3 V logic (D-51, D-53)"
+		(property "Description" "Board-to-board header. Unit 1: controller board (MCU, RJ45 LINK). Unit 2: EXP ribbon from the unit 1 controller board, +5V pins open at the controller end. 3.3 V logic (D-51, D-53). Samtec TSW, 0.64 mm square post 5.84 mm above the body, 10 uin gold on the post; mates with the ESQ-112-33-G-D on the controller (D-139)"
 			(at 314.96 198.12 0)
 			(hide yes)
+			(show_name no)
+			(do_not_autoplace no)
+			(effects
+				(font
+					(size 1.27 1.27)
+				)
+				(justify left)
+			)
+		)
+		(property "MPN" "TSW-112-07-L-D"
+			(at 314.96 198.12 0)
+			(hide yes)

Commit message: SO-239: 83-1R first source, 83-798 second (D-196, M-119)
Same flange, hole pattern, thread and front length (drawings 83-1R rev
AM, 83-798 rev AG). PBT insulator: solder the strap fast and check the
centre contact; no halogen statement (exception to D-135, reason
supply). Value and footprint unchanged; ERC 0; boards unchanged.

Co-Authored-By: Claude Opus 5.5 <noreply@anthropic.com>
Parts:
- J1, J10, J2, J3, J7, J8, J9: MPN 83-798 -> 83-1R
Changed lines of the file:
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@@
 		(company "PE1RGU - Shack Relay Matrix")
 		(comment 1 "Design: Prins Doornekamp, PE1RGU")
-		(comment 2 "RT1 RTD14012F x37, SO-239 Amphenol 83-798 x7, SMA EXP x3, XT60 x2, XT30")
+		(comment 2 "RT1 RTD14012F x37, SO-239 Amphenol 83-1R x7, SMA EXP x3, XT60 x2, XT30")
 		(comment 3 "Crossbar: rows on L1, columns on L6. Unit 1 = 3 radios x 4 antennas + EXP")
 		(comment 4 "JLC06161H-7628A, 1.6 mm, 6 layers. RF: CPWG W 0.975 / gap 2.0 mm, 50 ohm")
@@
 			)
 		)
-		(property "Description" "Radio R1. Amphenol RF 83-798 (SO-239/A, PTFE) in the case wall; strap to board pad"
+		(property "Description" "Radio R1. Amphenol RF 83-1R (SO-239, PBT insulator) in the case wall; strap to board pad. Second source Amphenol RF 83-798 (PTFE): same flange, holes and thread (D-196). PBT: solder the strap fast, check the centre contact after soldering"
 			(at 25.4 40.64 0)
 			(hide yes)
@@
 			)
 		)
-		(property "MPN" "83-798"
+		(property "MPN" "83-1R"
 			(at 25.4 40.64 0)
 			(hide yes)
@@
 			)
 		)
-		(property "Description" "Radio R2. Amphenol RF 83-798 (SO-239/A, PTFE) in the case wall; strap to board pad"
+		(property "Description" "Radio R2. Amphenol RF 83-1R (SO-239, PBT insulator) in the case wall; strap to board pad. Second source Amphenol RF 83-798 (PTFE): same flange, holes and thread (D-196). PBT: solder the strap fast, check the centre contact after soldering"
 			(at 25.4 101.6 0)
 			(hide yes)
@@
 			)
 		)
-		(property "MPN" "83-798"
+		(property "MPN" "83-1R"
 			(at 25.4 101.6 0)
 			(hide yes)
@@
 			)
 		)
-		(property "Description" "Radio R3. Amphenol RF 83-798 (SO-239/A, PTFE) in the case wall; strap to board pad"
+		(property "Description" "Radio R3. Amphenol RF 83-1R (SO-239, PBT insulator) in the case wall; strap to board pad. Second source Amphenol RF 83-798 (PTFE): same flange, holes and thread (D-196). PBT: solder the strap fast, check the centre contact after soldering"
 			(at 25.4 162.56 0)
 			(hide yes)
@@
 			)
 		)
-		(property "MPN" "83-798"
+		(property "MPN" "83-1R"
 			(at 25.4 162.56 0)
 			(hide yes)
@@
 			)
 		)
-		(property "Description" "Antenna A1. Amphenol RF 83-798 (SO-239/A, PTFE) in the case wall; strap to board pad"
+		(property "Description" "Antenna A1. Amphenol RF 83-1R (SO-239, PBT insulator) in the case wall; strap to board pad. Second source Amphenol RF 83-798 (PTFE): same flange, holes and thread (D-196). PBT: solder the strap fast, check the centre contact after soldering"
 			(at 279.4 40.64 0)
 			(hide yes)
@@
 			)
 		)
-		(property "MPN" "83-798"
+		(property "MPN" "83-1R"
 			(at 279.4 40.64 0)
 			(hide yes)
@@
 			)
 		)
-		(property "Description" "Antenna A2. Amphenol RF 83-798 (SO-239/A, PTFE) in the case wall; strap to board pad"
+		(property "Description" "Antenna A2. Amphenol RF 83-1R (SO-239, PBT insulator) in the case wall; strap to board pad. Second source Amphenol RF 83-798 (PTFE): same flange, holes and thread (D-196). PBT: solder the strap fast, check the centre contact after soldering"
 			(at 279.4 86.36 0)
 			(hide yes)
@@
 			)
 		)
-		(property "MPN" "83-798"
+		(property "MPN" "83-1R"
 			(at 279.4 86.36 0)
 			(hide yes)
@@
 			)
 		)
-		(property "Description" "Antenna A3. Amphenol RF 83-798 (SO-239/A, PTFE) in the case wall; strap to board pad"
+		(property "Description" "Antenna A3. Amphenol RF 83-1R (SO-239, PBT insulator) in the case wall; strap to board pad. Second source Amphenol RF 83-798 (PTFE): same flange, holes and thread (D-196). PBT: solder the strap fast, check the centre contact after soldering"
 			(at 279.4 132.08 0)
 			(hide yes)
@@
 			)
 		)
-		(property "MPN" "83-798"
+		(property "MPN" "83-1R"
 			(at 279.4 132.08 0)
 			(hide yes)
@@
 			)
 		)
-		(property "Description" "Antenna A4. Amphenol RF 83-798 (SO-239/A, PTFE) in the case wall; strap to board pad"
+		(property "Description" "Antenna A4. Amphenol RF 83-1R (SO-239, PBT insulator) in the case wall; strap to board pad. Second source Amphenol RF 83-798 (PTFE): same flange, holes and thread (D-196). PBT: solder the strap fast, check the centre contact after soldering"
 			(at 279.4 177.8 0)
 			(hide yes)
@@
 			)
 		)
-		(property "MPN" "83-798"
+		(property "MPN" "83-1R"
 			(at 279.4 177.8 0)
 			(hide yes)
