File: hardware/unit/rf-board/rf_detect.kicad_sch (KiCad schematic)
At the start: 17 parts, among them U801 LM2901

Commit message: Pre-order review; RF board seat keep-outs; part reuse P-1 to P-5
- docs/reviews/2026-10-31-pre-order-review.md: review of all three boards
  before ordering (verify scripts, ERC/DRC, pin maps, BOM, fab and case,
  firmware against spec, open items, part reuse).
- RF board (D-189, M-107): no other-net copper or vias under the case
  seats at S1 to S6 and the SO-239/SMA GND bosses; relay NC pads (pad 12)
  in netclass RF. Re-routed, DRC 0.
- Part reuse (D-190, M-108): one value text for 2k2, 100n 50V X7R and
  10n 50V X7R; shack PC817X order code as the controller; shack U4/U9 in
  VSSOP-8 (TI DCU, Nexperia DC) with fixed fan-out, re-routed.
  Netlists rf15, ctl15, si17; ERC 0.

Co-Authored-By: Claude Opus 5.5 <noreply@anthropic.com>
Parts:
- C801: value 100n -> 100n 50V X7R
Changed lines of the file:
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@@
 			)
 		)
-		(property "Value" "100n"
+		(property "Value" "100n 50V X7R"
 			(at 40.64 43.18 0)
 			(show_name no)

Commit message: S-6: order codes for LM2901, JST XH and shack 1 nF (M-117)
MPN fields only: RF U801 LM2901DR; shack J2/J7 B2B-XH-A(LF)(SN),
J6 B4B-XH-A(LF)(SN), 21 x 1 nF C0G GRM1885C1H102JA01D. Values,
netlists and boards unchanged. ERC 0 on both.

Co-Authored-By: Claude Opus 5.5 <noreply@anthropic.com>
Parts:
- U801: MPN LM2901 -> LM2901DR
Changed lines of the file:
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@@
 			)
 		)
-		(property "MPN" "LM2901"
+		(property "MPN" "LM2901DR"
 			(at 127.0 50.8 0)
 			(hide yes)
@@
 			)
 		)
-		(property "MPN" "LM2901"
+		(property "MPN" "LM2901DR"
 			(at 127.0 81.28 0)
 			(hide yes)
@@
 			)
 		)
-		(property "MPN" "LM2901"
+		(property "MPN" "LM2901DR"
 			(at 127.0 111.76 0)
 			(hide yes)
@@
 			)
 		)
-		(property "MPN" "LM2901"
+		(property "MPN" "LM2901DR"
 			(at 127.0 142.24 0)
 			(hide yes)
