File: hardware/unit/rf-board/power.kicad_sch (KiCad schematic)
At the start: 45 parts, among them Q1 PMV50EPEA, Q2 BSS138BK, U1 LP2985-33

Commit message: Pre-order review; RF board seat keep-outs; part reuse P-1 to P-5
- docs/reviews/2026-10-31-pre-order-review.md: review of all three boards
  before ordering (verify scripts, ERC/DRC, pin maps, BOM, fab and case,
  firmware against spec, open items, part reuse).
- RF board (D-189, M-107): no other-net copper or vias under the case
  seats at S1 to S6 and the SO-239/SMA GND bosses; relay NC pads (pad 12)
  in netclass RF. Re-routed, DRC 0.
- Part reuse (D-190, M-108): one value text for 2k2, 100n 50V X7R and
  10n 50V X7R; shack PC817X order code as the controller; shack U4/U9 in
  VSSOP-8 (TI DCU, Nexperia DC) with fixed fan-out, re-routed.
  Netlists rf15, ctl15, si17; ERC 0.

Co-Authored-By: Claude Opus 5.5 <noreply@anthropic.com>
Parts:
- C4: value 10n -> 10n 50V X7R
- R2: value 2.2k -> 2k2
Changed lines of the file:
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@@
 			)
 		)
-		(property "Value" "2.2k"
+		(property "Value" "2k2"
 			(at 80.01 68.58 0)
 			(show_name no)
@@
 			)
 		)
-		(property "Value" "10n"
+		(property "Value" "10n 50V X7R"
 			(at 119.38 127.0 0)
 			(show_name no)
@@
 			)
 		)
-		(property "Description" "LDO noise bypass, X7R or C0G"
+		(property "Description" "LDO noise bypass (one 10 nF line on all boards, D-190)"
 			(at 116.84 125.73 0)
 			(hide yes)

Commit message: S-4: MPN BSS138BK,215 (Nexperia) on RF and shack (M-115)
The ROHM BSS138BKT116 has the same name and another pin order. All 45
BSS138BK (RF 42, shack 3) now carry MPN BSS138BK,215. Nexperia pinning
1 G, 2 S, 3 D matches the footprint. ERC 0 on both; boards and
netlists unchanged.

Co-Authored-By: Claude Opus 5.5 <noreply@anthropic.com>
Parts:
- Q2: MPN BSS138BK -> BSS138BK,215
Changed lines of the file:
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@@
 			)
 		)
-		(property "MPN" "BSS138BK"
+		(property "MPN" "BSS138BK,215"
 			(at 78.74 78.74 0)
 			(hide yes)

Commit message: D-43 decided: clamp zener BZT52H-C24,115 (M-120)
Nexperia BZT52H-C24 passes the 13-coil clamp pulse (11.5 W peak, about
0.5 ms) against the PZSM curve (about 16 W at 0.5 ms). Diotec
BZT52C24 is the second source (no surge rating stated). Drain peak
39.1 V against 42 V. ERC 0; boards unchanged.

Co-Authored-By: Claude Opus 5.5 <noreply@anthropic.com>
Parts:
- D2, D3, D4, D5: MPN BZT52C24 -> BZT52H-C24,115
Changed lines of the file:
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@@
 			)
 		)
-		(property "Description" "Clamp zener, 24 V, SOD-123 (D-35, D-37): drain peak 12.6 + 24 + 0.9 = 37.5 V against 0.7 x 60 V. Part to confirm. Row and K1 coils"
+		(property "Description" "Clamp zener 24 V, SOD-123F on the SOD-123 land (D-35, D-37, D-43): drain peak 12.6 + 25.6 (VZ max) + 0.9 = 39.1 V against 0.7 x 60 V. Nexperia BZT52H-C24,115: PZSM about 16 W at 0.5 ms (Fig 1) against 11.5 W for 13 coils. Second source Diotec BZT52C24 (no surge rating stated). Row and K1 coils"
 			(at 139.7 67.31 0)
 			(hide yes)
@@
 			)
 		)
-		(property "MPN" "BZT52C24"
+		(property "MPN" "BZT52H-C24,115"
 			(at 139.7 67.31 0)
 			(hide yes)
@@
 			)
 		)
-		(property "Description" "Clamp zener, 24 V, SOD-123 (D-35, D-37): drain peak 12.6 + 24 + 0.9 = 37.5 V against 0.7 x 60 V. Part to confirm. Parallel to D2"
+		(property "Description" "Clamp zener 24 V, SOD-123F on the SOD-123 land (D-35, D-37, D-43): drain peak 12.6 + 25.6 (VZ max) + 0.9 = 39.1 V against 0.7 x 60 V. Nexperia BZT52H-C24,115: PZSM about 16 W at 0.5 ms (Fig 1) against 11.5 W for 13 coils. Second source Diotec BZT52C24 (no surge rating stated). Parallel to D2"
 			(at 154.94 67.31 0)
 			(hide yes)
@@
 			)
 		)
-		(property "MPN" "BZT52C24"
+		(property "MPN" "BZT52H-C24,115"
 			(at 154.94 67.31 0)
 			(hide yes)
@@
 			)
 		)
-		(property "Description" "Clamp zener, 24 V, SOD-123 (D-35, D-37): drain peak 12.6 + 24 + 0.9 = 37.5 V against 0.7 x 60 V. Part to confirm. K0 coils"
+		(property "Description" "Clamp zener 24 V, SOD-123F on the SOD-123 land (D-35, D-37, D-43): drain peak 12.6 + 25.6 (VZ max) + 0.9 = 39.1 V against 0.7 x 60 V. Nexperia BZT52H-C24,115: PZSM about 16 W at 0.5 ms (Fig 1) against 11.5 W for 13 coils. Second source Diotec BZT52C24 (no surge rating stated). K0 coils"
 			(at 40.64 101.6 0)
 			(hide yes)
@@
 			)
 		)
-		(property "MPN" "BZT52C24"
+		(property "MPN" "BZT52H-C24,115"
 			(at 40.64 101.6 0)
 			(hide yes)
@@
 			)
 		)
-		(property "Description" "Clamp zener, 24 V, SOD-123 (D-35, D-37): drain peak 12.6 + 24 + 0.9 = 37.5 V against 0.7 x 60 V. Part to confirm. Parallel to D3"
+		(property "Description" "Clamp zener 24 V, SOD-123F on the SOD-123 land (D-35, D-37, D-43): drain peak 12.6 + 25.6 (VZ max) + 0.9 = 39.1 V against 0.7 x 60 V. Nexperia BZT52H-C24,115: PZSM about 16 W at 0.5 ms (Fig 1) against 11.5 W for 13 coils. Second source Diotec BZT52C24 (no surge rating stated). Parallel to D3"
 			(at 55.88 101.6 0)
 			(hide yes)
@@
 			)
 		)
-		(property "MPN" "BZT52C24"
+		(property "MPN" "BZT52H-C24,115"
 			(at 55.88 101.6 0)
 			(hide yes)
